File: RAC-power.brd (EAGLE design)
At the start: 25.4 x 25.4 mm, 15 parts, among them J1 282834-2, U1 MCP1640, U2 TLA2022

Commit message: Fully routed board and cleared DRC
Parts:
- moved C3 13.0 mm to (3.30, 10.8), turned to 180 degrees
- moved U2 11.5 mm to (3.30, 13.5), turned to 180 degrees
- moved L1 5.09 mm to (13.1, 10.2)
- moved C2 5.08 mm to (13.1, 16.9), turned to 180 degrees
- moved R1 5.08 mm to (8.51, 14.5)
- moved R2 5.08 mm to (8.51, 16.1)
- moved U1 5.08 mm to (13.1, 14.0)
- moved C1 4.96 mm to (9.27, 11.4)
Routing:
- net V_BATT: track 0.00 -> 36.2 mm
- net VOUT: track 0.00 -> 20.3 mm
- net GND: track 0.00 -> 18.9 mm, vias 0 -> 6
- net SDA: track 0.00 -> 14.8 mm
- net SCL: track 0.00 -> 12.0 mm
- net EN: track 0.00 -> 5.26 mm
- net VFB: track 0.00 -> 4.31 mm
- added copper zone on layer 16, net GND
- added copper zone on layer 1, net SW
- added copper zone on layer 1, net V_BATT
